File: packages/kicad-parser/tests/demos/complex_hierarchy/ampli_ht.kicad_sch (KiCad schematic)
At the start: 29 parts, among them P201 CONN_2, P202 CONN_2, Q201 MPSA92, Q202 MPSA42, Q203 MPSA92, Q204 MPSA42, U201 LM358N

Commit message: FMT demos with 9.0x
Parts:
- added U1: OPA2836IRMCR, kicad_api_lib:OPA2836IRMCR, symbol OPA2836IRMCR:OPA2836IRMCR
