File: packages/kicad-parser/tests/demos/complex_hierarchy/complex_hierarchy.kicad_sch (KiCad schematic)
At the start: 10 parts, among them P101 CONN_2, P102 CONN_2, U101 78L05, U102 ICL7660

Commit message: FMT demos with 9.0x
Parts:
- added U3: OPA2836IRMCR, kicad_api_lib:OPA2836IRMCR, symbol OPA2836IRMCR:OPA2836IRMCR
