File: packages/kicad-parser/tests/demos/flat_hierarchy/flat_hierarchy.kicad_sch (KiCad schematic)
At the start: 0 parts

Commit message: FMT demos with 9.0x
Parts:
- added U7: LM6211MFX/NOPB, kicad_api_lib:LM6211MFX_NOPB, symbol LM6211MFX_NOPB:LM6211MFX_NOPB
