File: packages/kicad-parser/tests/demos/flat_hierarchy/pic_programmer.kicad_sch (KiCad schematic)
At the start: 56 parts, among them J1 DB9-FEMAL, P1 CONN_2, Q1 BC237, Q2 BC307, Q3 BC307, U2 74HC125, U3 7805, U4 LT1373

Commit message: FMT demos with 9.0x
Parts:
- added U9: LMC6042AIMX/NOPB, kicad_api_lib:LMC6042AIMX_NOPB, symbol LMC6042AIMX_NOPB:LMC6042AIMX_NOPB
