File: packages/kicad-parser/tests/demos/flat_hierarchy/pic_sockets.kicad_sch (KiCad schematic)
At the start: 8 parts, among them P2 SUPP28, P3 SUPP40, U1 24Cxx, U5 PIC_18_PINS, U6 PIC_8_PINS

Commit message: FMT demos with 9.0x
Parts:
- added U8: LM6211MFX/NOPB, kicad_api_lib:LM6211MFX_NOPB, symbol LM6211MFX_NOPB:LM6211MFX_NOPB
