File: packages/kicad-parser/tests/demos/video/bus_pci.kicad_sch (KiCad schematic)
At the start: 33 parts, among them U1 24C16, U11 S5933_PQ160

Commit message: FMT demos with 9.0x
Parts:
- added U26: TS1871IDT, kicad_api_lib:TS1871IDT, symbol TS1871IDT:TS1871IDT
