File: packages/kicad-parser/tests/demos/video/esvideo.kicad_sch (KiCad schematic)
At the start: 29 parts, among them U8 BT253, U9 BT473

Commit message: FMT demos with 9.0x
Parts:
- added U28: TS1871IDT, kicad_api_lib:TS1871IDT, symbol TS1871IDT:TS1871IDT
