File: packages/kicad-parser/tests/demos/video/graphic.kicad_sch (KiCad schematic)
At the start: 34 parts, among them P10 CONN_1, P11 CONN_1, P12 CONN_1, P4 CONN_2, P5 CONN_5, P9 CONN_1, U2 4C4001, U21 XC1736APD8, U23 XC4003/PQ100, U24 XC4005-PQ160, U7 AV9173, X1 10MHz

Commit message: FMT demos with 9.0x
Parts:
- added U27: TS1871IDT, kicad_api_lib:TS1871IDT, symbol TS1871IDT:TS1871IDT
