File: packages/kicad-parser/tests/demos/video/modul.kicad_sch (KiCad schematic)
At the start: 39 parts, among them Q1 BC848, Q2 BC848, Q3 BC848, U20 TDA8501, X3 4.433618MHz

Commit message: FMT demos with 9.0x
Parts:
- added U32: TS1871IDT, kicad_api_lib:TS1871IDT, symbol TS1871IDT:TS1871IDT
