File: packages/kicad-parser/tests/demos/video/muxdata.kicad_sch (KiCad schematic)
At the start: 5 parts, among them U22 XC4003-VQ100, U3 74LS245, U4 74LS245, U5 74LS245, U6 74LS245

Commit message: FMT demos with 9.0x
Parts:
- added U31: TS1871IDT, kicad_api_lib:TS1871IDT, symbol TS1871IDT:TS1871IDT
