File: packages/kicad-parser/tests/demos/video/pal-ntsc.kicad_sch (KiCad schematic)
At the start: 36 parts, among them U10 BT812, X2 30MHz

Commit message: FMT demos with 9.0x
Parts:
- added U29: TS1871IDT, kicad_api_lib:TS1871IDT, symbol TS1871IDT:TS1871IDT
