File: packages/kicad-parser/tests/demos/video/rams.kicad_sch (KiCad schematic)
At the start: 8 parts, among them U12 SIM4X32, U13 SIM4X32, U14 SIM4X32, U15 SIM4X32, U16 SIM4X32, U17 SIM4X32, U18 SIM4X32, U19 SIM4X32

Commit message: FMT demos with 9.0x
Parts:
- added U30: TS1871IDT, kicad_api_lib:TS1871IDT, symbol TS1871IDT:TS1871IDT
