File: packages/kicad-parser/tests/demos/video/video.kicad_sch (KiCad schematic)
At the start: 5 parts, among them J4 DB9FEM, P1 BNC, P2 BNC, P3 BNC, P8 BNC

Commit message: FMT demos with 9.0x
Parts:
- added U25: TS1871IDT, kicad_api_lib:TS1871IDT, symbol TS1871IDT:TS1871IDT
