File: packages/ecad-renderer/examples/mini-integration/assets/M5Pi.kicad_sch (KiCad schematic)
At the start: 141 parts, among them J1 Micro_SD_Card, J11 Grove_Socket_4Pin, J12 Conn_01x04, J2 Conn_02x15_Odd_Even, J3 Conn_01x02, J4 LCD_FPC_10P, J5 TOUCH_FPC_8P, J6 Speaker, Q1 Q_NMOS_GSD, SW1 Button_Tortoise_4Pin, SW2 Button_Tortoise_4Pin, U1 CH340E, U10 TP5400, U2 ESP8089, U3 F1C100s, U4 MPU-6050, U5 NS4158B, U6 SY8088AAC, U7 SY8088AAC, U8 SY8088AAC, U9 XC6206P302MR, Y1 26Mhz, Y2 24Mhz

Commit message: Update demo with cjk
Parts:
- removed AE1: Antenna_2.4G, imliubo-nightly:ANT-2.4GHZ-9.5X2.0MM, symbol imliubo-nightly:Antenna_2.4G
- removed C1, C10, C11, C12, C13, C14, C15, C17, C19, C2, C20, C21, C22, C23, C24, C27, C28, C29, C30, C44, C45, C47, C49, C50, C52, C53, C6, C7, C8, C9: 100nF, Capacitor_SMD:C_0402_1005Metric_Pad0.74x0.62mm_HandSolder, symbol Device:C
- removed C16: 10nF, Capacitor_SMD:C_0402_1005Metric_Pad0.74x0.62mm_HandSolder, symbol Device:C
- removed C18: 2.2nF, Capacitor_SMD:C_0402_1005Metric_Pad0.74x0.62mm_HandSolder, symbol Device:C
- removed C25, C26, C3, C4, C5, C57, Ci1: TBD, Capacitor_SMD:C_0402_1005Metric_Pad0.74x0.62mm_HandSolder, symbol Device:C
- removed C31, C33, C34, C35, C38, C39: 10uF, Capacitor_SMD:C_0603_1608Metric, symbol Device:C
- removed C32, C36, C37: 20pF, Capacitor_SMD:C_0603_1608Metric, symbol Device:C
- removed C40, C41, C46: 1uF, Capacitor_SMD:C_0402_1005Metric_Pad0.74x0.62mm_HandSolder, symbol Device:C
- removed C42, C43: 1uF, Capacitor_SMD:C_0603_1608Metric, symbol Device:C
- removed C48: 100uF, Capacitor_SMD:C_0402_1005Metric_Pad0.74x0.62mm_HandSolder, symbol Device:C
- removed C51: 10uF, Capacitor_SMD:C_0402_1005Metric_Pad0.74x0.62mm_HandSolder, symbol Device:C
- removed C54, C55: 22uF, Capacitor_SMD:C_0402_1005Metric_Pad0.74x0.62mm_HandSolder, symbol Device:C
- removed C56: C_Polarized, Capacitor_Tantalum_SMD:CP_EIA-3216-10_Kemet-I, symbol Device:C_Polarized
- removed D1: LED, LED_SMD:LED_0603_1608Metric_Pad1.05x0.95mm_HandSolder, symbol Device:LED
- removed D2, D3: LED, LED_SMD:LED_0402_1005Metric, symbol Device:LED
- removed D4: D, imliubo-nightly:D-SMA(DO-214AC), symbol Device:D
- removed D5: 1N5819, Diode_SMD:D_SOD-123, symbol Diode:1N5819
- removed F1: Fuse, Fuse:Fuse_1206_3216Metric, symbol Device:Fuse
- removed J1: Micro_SD_Card, imliubo-nightly:MicroSD_Socket_push, symbol imliubo-nightly:Micro_SD_Card
- removed J11: Grove_Socket_4Pin, imliubo-nightly:Grove_Socket_4Pin_2mm, symbol imliubo-nightly:Grove_Socket_4Pin
- removed J12: Conn_01x04, Connector_PinSocket_1.27mm:PinSocket_1x04_P1.27mm_Vertical, symbol Connector_Generic:Conn_01x04
- removed J2: Conn_02x15_Odd_Even, Connector_PinHeader_2.54mm:PinHeader_2x15_P2.54mm_Vertical, symbol Connector_Generic:Conn_02x15_Odd_Even
- removed J3: Conn_01x02, Connector_PinSocket_1.27mm:PinSocket_1x02_P1.27mm_Vertical, symbol Connector_Generic:Conn_01x02
- removed J4: LCD_FPC_10P, imliubo-nightly:TE_1-1734839-0_1x10-1MP_P0.5mm_Horizontal, symbol imliubo-nightly:CORE2_LCD_FPC_10P
- removed J5: TOUCH_FPC_8P, imliubo-nightly:TE_0-1734839-8_1x08-1MP_P0.5mm_Horizontal, symbol imliubo-nightly:CORE2_TOUCH_FPC_8P
- removed J6: Speaker, Connector_PinHeader_2.00mm:PinHeader_2x01_P2.00mm_Vertical, symbol Connector_Generic:Conn_01x02
- removed JP1: Jumper_3_Open, imliubo-nightly:SolderJumper-3_P1.3mm_Open_RoundedPad1.0x1.5mm, symbol Jumper:Jumper_3_Open
- removed L1, L2, L3: 2.2uH, Inductor_SMD:L_1008_2520Metric, symbol Device:L
- removed L4: 10uH, imliubo-nightly:L_Sunlord_SWPA4030S_4x4x3mm, symbol Device:L
- removed Q1: Q_NMOS_GSD, Package_TO_SOT_SMD:SOT-23, symbol Device:Q_NMOS_GSD
- removed R1: 1K, Resistor_SMD:R_0402_1005Metric, symbol Device:R
- removed R10, R3, R4, R9: 2K2, Resistor_SMD:R_0402_1005Metric_Pad0.72x0.64mm_HandSolder, symbol Device:R
- removed R11, R12, R13, R14, R15, R16, R27, R28, R29, R33, R39, R40, R41, R8: 10K, Resistor_SMD:R_0402_1005Metric_Pad0.72x0.64mm_HandSolder, symbol Device:R
- removed R17, R19, R36: 49K9, Resistor_SMD:R_0402_1005Metric_Pad0.72x0.64mm_HandSolder, symbol Device:R
- removed R18: 3K3, Resistor_SMD:R_0402_1005Metric_Pad0.72x0.64mm_HandSolder, symbol Device:R
- removed R2: 1.1K, Resistor_SMD:R_0402_1005Metric, symbol Device:R
- removed R20: 5.1K, Resistor_SMD:R_0402_1005Metric_Pad0.72x0.64mm_HandSolder, symbol Device:R
- removed R21: 680K, Resistor_SMD:R_0402_1005Metric, symbol Device:R
- removed R22, R24, R25, R26: 150K, Resistor_SMD:R_0402_1005Metric, symbol Device:R
- removed R23: 470K, Resistor_SMD:R_0402_1005Metric, symbol Device:R
- removed R30, R31: 200K, Resistor_SMD:R_0402_1005Metric_Pad0.72x0.64mm_HandSolder, symbol Device:R
- removed R32, R37, R6, R7: 4.7K, Resistor_SMD:R_0402_1005Metric_Pad0.72x0.64mm_HandSolder, symbol Device:R
- removed R34, R35, Ri1: TBD, Resistor_SMD:R_0402_1005Metric_Pad0.72x0.64mm_HandSolder, symbol Device:R
- removed R5: 12K, Resistor_SMD:R_0402_1005Metric_Pad0.72x0.64mm_HandSolder, symbol Device:R
- removed SW1, SW2: Button_Tortoise_4Pin, imliubo-nightly:Button_4Pin_Tortoise, symbol imliubo-nightly:Button_Tortoise_4Pin
- removed TBD1: L, Inductor_SMD:L_0402_1005Metric_Pad0.77x0.64mm_HandSolder, symbol Device:L
- removed TP1, TP2, TP3, TP4, TP5: TestPoint, imliubo-nightly:TestPoint, symbol imliubo-nightly:TestPoint
- removed U1: CH340E, Package_SO:MSOP-10_3x3mm_P0.5mm, symbol Interface_USB:CH340E
- removed U10: TP5400, imliubo-nightly:SOP-8_4.8x6.0mm_P1.27mm_EP2.3x3.2mm, symbol imliubo-nightly:TP5400
- removed U2: ESP8089, Package_DFN_QFN:QFN-32-1EP_5x5mm_P0.5mm_EP3.45x3.45mm, symbol imliubo-nightly:ESP8089
- removed U3: F1C100s, imliubo-nightly:QFN-88_EP_10x10_Pitch0.4mm, symbol imliubo-nightly:F1C100s
- removed U4: MPU-6050, Sensor_Motion:InvenSense_QFN-24_4x4mm_P0.5mm, symbol Sensor_Motion:MPU-6050
- removed U5: NS4158B, imliubo-nightly:SOP-8_3.9x4.9mm_P1.27mm, symbol imliubo-nightly:NS4158B
- removed U6, U7, U8: SY8088AAC, Package_TO_SOT_SMD:SOT-23-5, symbol imliubo-nightly:SY8088AAC
- removed U9: XC6206P302MR, Package_TO_SOT_SMD:SOT-23, symbol Regulator_Linear:XC6206PxxxMR
- removed UART1: USB_C, imliubo-nightly:USB_C_C393939, symbol imliubo-nightly:USB_C
- removed Y1: 26Mhz, Crystal:Crystal_SMD_3225-4Pin_3.2x2.5mm, symbol Device:Crystal_GND24
- removed Y2: 24Mhz, Crystal:Crystal_SMD_3225-4Pin_3.2x2.5mm, symbol Device:Crystal_GND24
- added Q1: NCE30P50G, kicad_api_lib:NCE30P50G, symbol NCE30P50G:NCE30P50G
- added Q2: 2N7002Q-7-F, kicad_api_lib:2N7002Q-7-F, symbol 2N7002Q-7-F:2N7002Q-7-F
- added R1, R2: 10K, kicad_api_lib:AC0402FR-0710KL, symbol AC0402FR-0710KL:AC0402FR-0710KL
- added R3: 300K, kicad_api_lib:AC0402FR-07300KL, symbol AC0402FR-07300KL:AC0402FR-07300KL
Connections:
- net GND: now also Q2.3 (S), R3.2
- new net: Q1.4 (G), R1.2, R2.1
- new net: Q2.2 (D), R2.2
- new net CTRL: Q2.1 (G), R3.1
- new net PWR_IN: Q1.1 (S), Q1.2 (S), Q1.3 (S), R1.1
- new net PWR_OUT: Q1.5 (D), Q1.6 (D), Q1.7 (D), Q1.8 (D), Q1.9 (D)
- no-connect marks 32 -> 0
Other:
- note added: "NCE30P50G_MOS Electronic Switch"
- note added: "模块电路功能： 这是一个基于 P 沟道 MOSFET 的高边电源开关电路， 核心作用是用低电压控制信号控制主电源向负载的供电通断。 CTRL为高电平时，Q2导通，将Q1栅极拉低，从而使Q1导通，PWR_IN正常输出； CTRL为低电平时，Q2关断，Q1关断，PWR_IN信号无法输出。 引脚功能： CTRL：低电压数字信号，控制输入电源（PWR_IN）向负载（PWR_OUT）的通断； 供电电压： PWR_IN：输入电源，2V-24V； PWR_OUT：输出电源； 应用场景： 单片机 / MCU 控制的外设供电开关、便携设备、移动电源、锂电池组的供电通断控制、 小家电的电源控制、USB 设备的供电开关。"
- note removed: "6V 2A"
- note removed: "AMP"
- note removed: "Audio"
- note removed: "C113101"
- note removed: "CPU"
- note removed: "CPU Power"
- note removed: "Designer By IAMLIUBO CC BY-NC-ND 4.0"
- note removed: "GPIO"
- note removed: "I2C"
- note removed: "I2C0"
- note removed: "I2C1"
- note removed: "I2C2"
- note removed: "I2S"
- note removed: "LCD"
- note removed: "LCD SPI1"
- note removed: "M-BUS"
- note removed: "MPU I2C0"
- note removed: "On Board"
- note removed: "Power"
- note removed: "R1"
- note removed: "R2"
- note removed: "RESET KEY & LED"
- note removed: "SPI"
- note removed: "TF-Card"
- note removed: "UART"
- note removed: "USART1"
- note removed: "USART2"
- note removed: "USB"
- note removed: "VCTRL 0.4VDD - VDD 普通模式 0.9V - 0.4VDD 防失真模式 0 - 0.2V ShutDown"
- note removed: "Wi-Fi SPI0"
- title: M5Pi-F1C100S/200S -> (none)
